File: pressure_trigger_pcb_project/ABP_Trigger_Board/first_draft_schematic.brd (EAGLE design)
At the start: 67.6 x 33 mm, 28 parts, among them U1 OPA4340UA

Commit message: schematic before package switch
Parts:
- removed LED: WIREPAD1,6/0,9, wirepad:1,6/0,9
- added L1, L2, LED2, PAD1, PAD2: WIREPAD1,6/0,9, wirepad:1,6/0,9
- added R10, R11: 681, resistor:R0805
- moved SEL 12.8 mm to (23.5, 26.0)
- moved MRI 12.8 mm to (27.3, 26.0)
- moved PAD7 8.91 mm to (23.5, 29.2)
- moved PAD8 8.91 mm to (27.3, 29.2)
- moved R9 3.14 mm to (21.9, 23.8), turned to 0 degrees
- moved DH 1.59 mm to (8.26, 26.0)
- moved PAD6 1.42 mm to (12.1, 29.2)
- moved TC 0.64 mm to (64.8, 18.4)
- moved TG 0.63 mm to (64.8, 14.6)
- moved SG 0.63 mm to (64.8, 22.2)
- renumbered TEENSY3.0 to TEENSY3.0-MICROCONTROLLER
Connections:
- new net N$18: L1.1, R10.1
- new net N$21: R10.2, TEENSY3.0-MICROCONTROLLER.19/A5
- new net N$22: LED2.1, R11.1
- new net N$23: R11.2, TEENSY3.0-MICROCONTROLLER.20/A6
- net GND: now also PAD1.1, PAD2.1
- net N$11: now also L2.1; no longer LED.1
- net N$14: now also TEENSY3.0-MICROCONTROLLER.18/A4; no longer TEENSY3.0-MICROCONTROLLER.16/A2
- net N$15: now also TEENSY3.0-MICROCONTROLLER.16/A2; no longer TEENSY3.0-MICROCONTROLLER.17/A3
- net N$16: now also TEENSY3.0-MICROCONTROLLER.17/A3; no longer TEENSY3.0-MICROCONTROLLER.18/A4
Routing:
- net N$16: track 15.9 -> 7.40 mm
- net N$23: track 0.00 -> 7.43 mm
- net N$15: track 13.5 -> 6.88 mm
- net N$21: track 0.00 -> 5.44 mm
- net N$11: track 6.64 -> 2.75 mm
- net N$14: track 7.24 -> 4.39 mm
- net N$22: track 0.00 -> 2.75 mm
- net N$18: track 0.00 -> 2.22 mm
- net N$13: track 3.91 -> 4.68 mm
- net N$5: track 17.9 -> 17.3 mm
- net VCC: track 147.7 -> 148.3 mm
Other:
- board text added: "AD5206UABR50"
- board text added: "OPA4340"
- board text removed: "ARTERIAL BP TRIGGERING SYSTEM REV B JOSHBRADSHAW11@GMAIL.COM"

Commit message: finalized board layout
Parts:
- removed AD5206-50: AD5206BRUZ10, AD5206:SOP65P640X120-24N
- added U2: AD5206BRUZ10SOIC24R, AD5206_SOIC:SO24R
- moved C2 3.42 mm to (40.0, 8.26), turned to 0 degrees
- turned R8 to 0 degrees
Connections:
- net GND: now also U2.4, U2.9; no longer AD5206-50.4, AD5206-50.9
- net N$12: now also U2.14; no longer AD5206-50.14
- net N$17: now also U2.13; no longer AD5206-50.13
- net N$19: now also U2.8; no longer AD5206-50.8
- net N$3: now also U2.23; no longer AD5206-50.23
- net N$5: now also U2.24; no longer AD5206-50.24
- net N$7: now also U2.5; no longer AD5206-50.5
- net N$8: now also U2.7; no longer AD5206-50.7
- net VCC: now also U2.6; no longer AD5206-50.6
Routing:
- net VCC: track 148.3 -> 155.5 mm
- net GND: track 21.1 -> 27.8 mm
- net AGND: track 18.7 -> 13.7 mm
- net N$8: track 20.3 -> 25.2 mm
- net N$7: track 22.0 -> 25.9 mm
- net N$19: track 27.0 -> 30.6 mm
- net N$17: track 18.1 -> 17.1 mm
- net N$9: track 26.7 -> 27.5 mm
- net N$2: track 30.8 -> 31.6 mm
- net N$5: track 17.3 -> 16.6 mm
- net N$10: track 17.3 -> 17.8 mm
Other:
- board size 67.6 x 33 mm -> 68.6 x 37.5 mm
- board text added: "Arterial BP Triggering System REV B Josh Bradshaw, 2015"
- board text removed: "AD5206UABR50"
